File: Sofle_v2/PCB/SofleKeyboard.kicad_pcb (KiCad board)
At the start: 2 copper layers, 143.5 x 115.5 mm, 89 parts, among them J1 LED, J2 4PIN, J3 OLED, SW1 SW_PUSH, SW10 SW_PUSH, SW11 SW_PUSH, SW12 SW_PUSH, SW13 SW_PUSH, SW14 SW_PUSH, SW15 SW_PUSH, SW16 SW_PUSH, SW17 SW_PUSH, SW18 SW_PUSH, SW19 SW_PUSH, SW2 SW_PUSH, SW20 SW_PUSH, SW21 SW_PUSH, SW22 SW_PUSH, SW23 SW_PUSH, SW24 SW_PUSH, SW25 Rotary_Encoder_Switch, SW26 SW_PUSH, SW27 SW_PUSH, SW28 SW_PUSH, SW29 SW_PUSH, SW3 SW_PUSH, SW30 SW_PUSH, SW4 SW_PUSH, SW5 SW_PUSH, SW6 SW_PUSH, SW7 SW_PUSH, SW8 SW_PUSH, SW9 SW_PUSH, U1 ProMicro

Commit message: initial prototype
Parts:
- removed D25: D, SofleKeyboard-footprint:Diode_SOD123
- removed J2: 4PIN, SofleKeyboard-footprint:MJ-4PP-9
- removed J3: OLED, SofleKeyboard-footprint:OLED_4Pin
- removed JP1, JP2, JP3, JP4, JP5, JP6, JP7, JP8: Jumper_NO_Small, SofleKeyboard-footprint:Jumper
- removed JP10: IC2SDA, Jumper:SolderJumper-2_P1.3mm_Open_TrianglePad1.0x1.5mm
- removed JP11: Serial, Jumper:SolderJumper-2_P1.3mm_Bridged2Bar_Pad1.0x1.5mm
- removed JP9: I2CSCL, Jumper:SolderJumper-2_P1.3mm_Open_TrianglePad1.0x1.5mm
- removed R1, R2: R, SofleKeyboard-footprint:R_1206_DoubleSided
- removed RSW1: SW_RST, SofleKeyboard-footprint:TACT_SWITCH_TVBP06
- removed TH1, TH2: HOLE, SofleKeyboard-footprint:M2_HOLE_PCB
- added G***: LOGO, xenia:xenia, F.Cu at (98.1, 70.4)
- added G***: LOGO, xenia:xenia, B.Cu at (98.1, 70.4)
- D1, D10, D11, D12, D13, D14, D15, D16, D17, D18, D19, D2, D20, D21, D22, D23, D24, D26, D27, D28, D29, D3, D30, D4, D5, D6, D7, D8, D9: footprint SofleKeyboard-footprint:Diode_SOD123 -> custom:D_SOD-123_flip
- J1: value LED -> Conn_01x02; footprint SofleKeyboard-footprint:LED -> custom:Battery
- SW25: value Rotary_Encoder_Switch -> SW_DPDT_x2; footprint SofleKeyboard-footprint:RotaryEncoder_Alps_EC11E-Switch_Vertical_H20mm-keebio_modified -> custom:MSK-12C02_DUAL
- U1: value ProMicro -> XIAO_nRF52840; footprint SofleKeyboard-footprint:ArduinoProMicro-ZigZag-DoubleSided -> custom:XIAO_nRF52840_DUAL
- moved SW25 41.2 mm to (84.3, 68.1), turned to 90 degrees
- moved J1 26.2 mm to (97.3, 79.4), turned to 180 degrees
- moved U1 16.2 mm to (96.7, 40.8), turned to 0 degrees
Connections:
- J1 pad 1: VCC -> +BATT
- J1 pad 2: LED -> batt_alt
- SW1 pad 1: SW25A -> col5
- SW13 pad 1: SW25A -> col5
- SW19 pad 1: SW25A -> col5
- SW26 pad 1: col4 -> col5
- SW27 pad 1: col3 -> col4
- SW28 pad 1: col2 -> col3
- SW29 pad 1: col1 -> col2
- SW30 pad 1: col0 -> col1
- SW7 pad 1: SW25A -> col5
- U1 pad 1: LED -> col0
- U1 pad 10: row2 -> col3
- U1 pad 11: row3 -> col2
- U1 pad 12: row4 -> unconnected-(U1-3V3-Pad12)
- U1 pad 13: SW25A -> GND
- U1 pad 14: col4 -> unconnected-(U1-5V-Pad14)
- U1 pad 19: ENCB -> +BATT
- U1 pad 2: DATA -> col1
- U1 pad 20: ENCA -> -BATT
- U1 pad 3: GND -> row0
- U1 pad 4: GND -> row1
- U1 pad 5: SDA -> row2
- U1 pad 6: SCL -> row3
- U1 pad 7: (no net) -> row4
- U1 pad 8: row0 -> col5
- U1 pad 9: row1 -> col4
Routing:
- net col5: track 0.00 -> 130.6 mm, vias 0 -> 6
- net GND: track 122.6 -> 0.00 mm, vias 73 -> 0
- net SW25A: track 103.3 -> 0.00 mm, vias 5 -> 0
- net VCC: track 90.9 -> 0.00 mm, vias 3 -> 0
- net ENCB: track 61.9 -> 0.00 mm
- net LED: track 60.2 -> 0.00 mm, vias 1 -> 0
- net ENCA: track 57.8 -> 0.00 mm
- net RESET: track 43.2 -> 0.00 mm
- net +BATT: track 0.00 -> 42.5 mm, vias 0 -> 1
- net -BATT: track 0.00 -> 36.6 mm, vias 0 -> 2
- net SDA: track 36.0 -> 0.00 mm, vias 2 -> 0
- net /i2c_d: track 35.7 -> 0.00 mm, vias 1 -> 0
- net SCL: track 33.5 -> 0.00 mm, vias 2 -> 0
- net col0: track 229.8 -> 198.1 mm
- net /i2c_c: track 30.5 -> 0.00 mm, vias 2 -> 0
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- removed copper zone on B.Cu, net GND
- removed copper zone on F.Cu, net GND
Other:
- outline, holes or cut-outs redrawn
- net class Default removed
- net class GND removed
- net class VCC removed
- rule pad_to_mask_clearance: 0.2 -> 0
